File: my-own-keyboard.kicad_pcb (KiCad board)
At the start: 2 copper layers, 285.8 x 95.2 mm, 140 parts, among them J2 5077CR-16SMC2-BK-TR, SW1 Reset SW, SW10 8, SW11 9, SW12 0, SW13 -, SW14 =, SW15 Backspace, SW16 Tab, SW17 Q, SW18 W, SW19 E, SW2 `, SW20 R, SW21 T, SW22 Y, SW23 U, SW24 I, SW25 O, SW26 P, SW27 [, SW28 ], SW29 \, SW3 1, SW30 Capslock, SW31 A, SW32 S, SW33 D, SW34 F, SW35 G, SW36 H, SW37 J, SW38 K, SW39 L, SW4 2, SW40 ;, SW41 ', SW42 Enter, SW43 L-shift, SW44 Z, SW45 X, SW46 C, SW47 V, SW48 B, SW49 N, SW5 3, SW50 M, SW51 ,, SW52 ., SW53 /, SW54 R-shift, SW55 L-Ctrl, SW56 win, SW57 L-Alt, SW58 Space, SW59 Fn, SW6 4, SW60 R-Alt, SW61 Menu, SW62 R-Ctrl, SW63 RotaryEncoder_Switch, SW7 5, SW8 6, SW9 7, U1 ATmega32U4-A, Y1 16MHz

Commit message: wired
Parts:
- moved C1 2.31 mm to (339.2, 139.7)
- moved C7 0.89 mm to (342.4, 139.7)
- moved C6 0.55 mm to (342.4, 137.0)
- moved C4 0.43 mm to (342.4, 134.1)
- turned SW1 to 90 degrees
Connections:
- C4 pad 1: RESET -> VCC
- C5 pad 1: RESET -> VCC
- C6 pad 1: RESET -> VCC
- C7 pad 1: RESET -> VCC
- J2 pad A4_B9: RESET -> VCC
- J2 pad B4_A9: RESET -> VCC
- SW1 pad 1: RESET -> GND
- SW1 pad 2: GND -> VCC
- U1 pad 13: RESET -> VCC
- U1 pad 14: RESET -> VCC
- U1 pad 2: RESET -> VCC
- U1 pad 24: RESET -> VCC
- U1 pad 34: RESET -> VCC
- U1 pad 44: RESET -> VCC
- U1 pad 7: RESET -> VCC
Routing:
- net row0: track 0.00 -> 294.3 mm
- net row1: track 0.00 -> 289.8 mm
- net row4: track 0.00 -> 285.3 mm
- net row2: track 0.00 -> 275.5 mm
- net row3: track 0.00 -> 258.9 mm
- net GND: track 0.00 -> 166.2 mm
- net VCC: track 0.00 -> 132.7 mm, vias 0 -> 6
- net col2: track 0.00 -> 96.6 mm
- net col1: track 0.00 -> 95.7 mm
- net col12: track 0.00 -> 95.3 mm
- net col3: track 0.00 -> 90.1 mm
- net col6: track 0.00 -> 90.0 mm
- net col9: track 0.00 -> 89.2 mm
- net col0: track 0.00 -> 87.9 mm
- net col11: track 0.00 -> 87.0 mm
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
Commit message: completed wiring
Parts:
- moved D41 2.45 mm to (330.9, 137.2)
- moved C5 1.10 mm to (349.9, 147.2)
Connections:
- U1 pad 1: unconnected-(U1-PE6-Pad1) -> row0
- U1 pad 10: unconnected-(U1-PB2-Pad10) -> MOSI
- U1 pad 11: unconnected-(U1-PB3-Pad11) -> MISO
- U1 pad 18: unconnected-(U1-PD0-Pad18) -> RE_A
- U1 pad 19: unconnected-(U1-PD1-Pad19) -> RE_B
- U1 pad 20: unconnected-(U1-PD2-Pad20) -> col0
- U1 pad 21: unconnected-(U1-PD3-Pad21) -> col1
- U1 pad 22: unconnected-(U1-PD5-Pad22) -> col2
- U1 pad 25: unconnected-(U1-PD4-Pad25) -> col3
- U1 pad 26: unconnected-(U1-PD6-Pad26) -> col4
- U1 pad 27: unconnected-(U1-PD7-Pad27) -> col5
- U1 pad 28: unconnected-(U1-PB4-Pad28) -> col6
- U1 pad 29: unconnected-(U1-PB5-Pad29) -> col7
- U1 pad 30: unconnected-(U1-PB6-Pad30) -> col10
- U1 pad 31: unconnected-(U1-PC6-Pad31) -> col9
- U1 pad 32: unconnected-(U1-PC7-Pad32) -> col8
- U1 pad 36: unconnected-(U1-PF7-Pad36) -> row4
- U1 pad 37: unconnected-(U1-PF6-Pad37) -> row3
- U1 pad 38: unconnected-(U1-PF5-Pad38) -> col11
- U1 pad 39: unconnected-(U1-PF4-Pad39) -> col12
- U1 pad 40: unconnected-(U1-PF1-Pad40) -> row2
- U1 pad 41: unconnected-(U1-PF0-Pad41) -> row1
- U1 pad 8: unconnected-(U1-PB0-Pad8) -> col13
- U1 pad 9: unconnected-(U1-PB1-Pad9) -> SCK
Routing:
- net col0: track 87.9 -> 387.3 mm
- net col2: track 96.6 -> 340.7 mm
- net col1: track 95.7 -> 303.3 mm
- net col3: track 90.1 -> 294.3 mm
- net col4: track 67.0 -> 271.0 mm, vias 0 -> 1
- net col5: track 67.0 -> 252.8 mm, vias 0 -> 1
- net col6: track 90.0 -> 234.1 mm
- net col7: track 67.2 -> 208.5 mm, vias 0 -> 1
- net col8: track 67.0 -> 177.8 mm, vias 0 -> 1
- net col9: track 89.2 -> 179.3 mm
- net col10: track 87.0 -> 155.0 mm
- net col13: track 21.0 -> 63.4 mm, vias 0 -> 1
- net col11: track 87.0 -> 126.4 mm, vias 0 -> 1
- net XTAL2: track 3.28 -> 31.8 mm, vias 0 -> 2
- net row0: track 294.3 -> 321.4 mm, vias 0 -> 1
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
Commit message: added ICSP
Parts:
- added ICSP: ICSP, Connector_PinSocket_1.27mm:PinSocket_2x03_P1.27mm_Vertical, F.Cu at (350.8, 167.2)
- added R6: 10k, Resistor_SMD:R_0603_1608Metric, B.Cu at (349.1, 94.6)
- turned SW1 to -90 degrees
Connections:
- SW1 pad 1: GND -> Reset
- SW1 pad 2: VCC -> GND
- U1 pad 13: VCC -> Reset
Routing:
- net Reset: track 0.00 -> 89.1 mm, vias 0 -> 2
- net MOSI: track 0.00 -> 33.0 mm, vias 0 -> 1
- net MISO: track 0.00 -> 27.2 mm, vias 0 -> 1
- net SCK: track 0.00 -> 26.0 mm, vias 0 -> 1
- net VCC: track 131.7 -> 143.1 mm, vias 7 -> 9
- net GND: track 179.5 -> 185.6 mm
- net XTAL1: track 26.3 -> 25.6 mm
- added copper zone on B.Cu, net GND
- added copper zone on F.Cu, net GND

Commit message: completed all of the design of the PCB
Parts:
- added G***: LOGO, logo:logo-mini, F.Cu at (314.8, 128.4)
- added G***: LOGO, logo:logo-mini, B.Cu at (314.8, 128.4)
Routing:
- net SCK: track 26.0 -> 33.3 mm
- net MOSI: track 33.0 -> 27.7 mm
- net VCC: track 143.1 -> 141.8 mm
- net Reset: track 89.1 -> 89.8 mm

Commit message: created the holes
Parts:
- added REF**: MountingHole_2.2mm_M2, MountingHole:MountingHole_2.2mm_M2, F.Cu at (195.3, 164.3)
- added REF**: MountingHole_2.2mm_M2, MountingHole:MountingHole_2.2mm_M2, F.Cu at (209.6, 119.1)
- added REF**: MountingHole_2.2mm_M2, MountingHole:MountingHole_2.2mm_M2, F.Cu at (309.6, 150.0)
- added REF**: MountingHole_2.2mm_M2, MountingHole:MountingHole_2.2mm_M2, F.Cu at (92.9, 109.5)
- added REF**: MountingHole_2.2mm_M2, MountingHole:MountingHole_2.2mm_M2, F.Cu at (326.2, 109.5)
- added REF**: MountingHole_2.2mm_M2, MountingHole:MountingHole_2.2mm_M2, F.Cu at (71.4, 152.4)
- moved D21 3.17 mm to (201.6, 118.3)
Routing:
- net col1: track 303.3 -> 373.6 mm
- net col0: track 387.3 -> 394.2 mm
- net row4: track 298.4 -> 304.5 mm
- net col2: track 340.7 -> 342.9 mm
- net col4: track 271.0 -> 273.2 mm
- net col3: track 294.3 -> 296.2 mm
- net col5: track 252.8 -> 254.3 mm
- net Net-(D21-A): track 17.9 -> 19.2 mm
- net col6: track 234.1 -> 235.2 mm
- net row1: track 296.9 -> 298.1 mm

Commit message: updated the pcb
Parts:
- removed G*** (x2): LOGO, logo:logo-mini
- removed the REF** at (195.3, 164.3)
- removed the REF** at (209.6, 119.1)
- removed the REF** at (309.6, 150.0)
- removed the REF** at (92.9, 109.5)
- removed the REF** at (326.2, 109.5)
- removed the REF** at (71.4, 152.4)
- added REF**: Stabilizer, BrownSugar_KBD:Stabilizer_MX_PCB_Mount_3U, F.Cu at (223.8, 166.7)
- added REF**: Stabilizer, BrownSugar_KBD:Stabilizer_MX_PCB_Mount_3U, F.Cu at (166.7, 166.7)
- added REF**: Stabilizer, BrownSugar_KBD:Stabilizer_MX_PCB_Mount_2U, F.Cu at (333.4, 90.5)
- added REF**: Stabilizer, BrownSugar_KBD:Stabilizer_MX_PCB_Mount_2U, F.Cu at (331.0, 128.6)
- added REF**: Stabilizer, BrownSugar_KBD:Stabilizer_MX_PCB_Mount_2U, F.Cu at (88.1, 147.6)
- added REF**: Stabilizer, BrownSugar_KBD:Stabilizer_MX_PCB_Mount_2U, F.Cu at (326.2, 147.6)
- Reset: renamed from SW1; footprint kbd:ResetSW -> original_library:ResetSW TSHA-T-2.5B2-19SH
- moved Reset 255.1 mm to (95.2, 118.1), turned to 0 degrees
- moved J2 232.8 mm to (85.7, 85.7)
- moved U1 147.9 mm to (195.3, 166.7), turned to 180 degrees
- moved R3 59.1 mm to (375.7, 99.2)
- moved R5 59.1 mm to (381.6, 100.0)
- moved R2 59.1 mm to (378.5, 99.2)
- moved R4 59.1 mm to (379.6, 102.5)
- moved R1 45.2 mm to (381.6, 150.4)
- moved C1 37.1 mm to (376.1, 136.1)
- moved C4 37.1 mm to (379.3, 130.5)
- moved C6 37.1 mm to (379.3, 133.3)
- moved C7 37.1 mm to (379.3, 136.1)
- moved J1 31.3 mm to (381.5, 161.1)
- moved R6 30.2 mm to (379.2, 92.8)
- moved C5 28.7 mm to (377.7, 140.0)
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- renumbered ICSP to J1
Routing:
- net col0: track 394.2 -> 0.00 mm
- net col1: track 373.6 -> 0.00 mm
- net col2: track 342.9 -> 0.00 mm
- net row0: track 321.4 -> 0.00 mm, vias 1 -> 0
- net row4: track 304.5 -> 0.00 mm, vias 1 -> 0
- net row1: track 298.1 -> 0.00 mm
- net col3: track 296.2 -> 0.00 mm
- net col4: track 273.2 -> 0.00 mm, vias 1 -> 0
- net row2: track 260.7 -> 0.00 mm
- net col5: track 254.3 -> 0.00 mm, vias 1 -> 0
- net row3: track 248.3 -> 0.00 mm
- net col6: track 235.2 -> 0.00 mm
- net col7: track 208.5 -> 0.00 mm, vias 1 -> 0
- net GND: track 185.6 -> 0.00 mm, vias 2 -> 0
- net col9: track 179.3 -> 0.00 mm
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- removed copper zone on B.Cu, net GND
- removed copper zone on F.Cu, net GND
