File: my-own-keyboard.kicad_pcb (KiCad board)
At the start: 2 copper layers, 285.8 x 95.2 mm, 148 parts, among them J1 ICSP, J2 5077CR-16SMC2-BK-TR, SW10 8, SW11 9, SW12 0, SW13 -, SW14 =, SW15 Backspace, SW16 Tab, SW17 Q, SW18 W, SW19 E, SW2 `, SW20 R, SW21 T, SW22 Y, SW23 U, SW24 I, SW25 O, SW26 P, SW27 [, SW28 ], SW29 \, SW3 1, SW30 Capslock, SW31 A, SW32 S, SW33 D, SW34 F, SW35 G, SW36 H, SW37 J, SW38 K, SW39 L, SW4 2, SW40 ;, SW41 ', SW42 Enter, SW43 L-shift, SW44 Z, SW45 X, SW46 C, SW47 V, SW48 B, SW49 N, SW5 3, SW50 M, SW51 ,, SW52 ., SW53 /, SW54 R-shift, SW55 L-Ctrl, SW56 win, SW57 L-Alt, SW58 Space, SW59 Fn, SW6 4, SW60 R-Alt, SW61 Menu, SW62 R-Ctrl, SW63 RotaryEncoder_Switch, SW7 5, SW8 6, SW9 7, U1 ATmega32U4-A, Y1 16MHz

Commit message: updated the directory
Parts:
- D1, D10, D11, D12, D13, D14, D15, D16, D17, D18, D19, D2, D20, D21, D22, D23, D24, D25, D26, D27, D28, D29, D3, D30, D31, D32, D33, D34, D35, D36, D37, D38, D39, D4, D40, D41, D42, D43, D44, D45, D46, D47, D48, D49, D5, D50, D51, D52, D53, D54, D55, D56, D57, D58, D59, D6, D60, D61, D62, D7, D8, D9: footprint kbd:D3_TH_SMD -> others:D3_TH_SMD
- SW10, SW11, SW12, SW13, SW14, SW17, SW18, SW19, SW2, SW20, SW21, SW22, SW23, SW24, SW25, SW26, SW27, SW28, SW3, SW31, SW32, SW33, SW34, SW35, SW36, SW37, SW38, SW39, SW4, SW40, SW41, SW44, SW45, SW46, SW47, SW48, SW49, SW5, SW50, SW51, SW52, SW53, SW6, SW7, SW8, SW9: footprint BrownSugar_KBD:CherryMX_Hotswap_via_1U -> keyswitch:CherryMX_Hotswap_via_1U
- SW15: footprint BrownSugar_KBD:CherryMX_Hotswap_via_2U -> keyswitch:CherryMX_Hotswap_via_2U
- SW16, SW29: footprint BrownSugar_KBD:CherryMX_Hotswap_via_1.5U -> keyswitch:CherryMX_Hotswap_via_1.5U
- SW30: footprint BrownSugar_KBD:CherryMX_Hotswap_via_1.75U -> keyswitch:CherryMX_Hotswap_via_1.75U
- SW42, SW43: footprint BrownSugar_KBD:CherryMX_Hotswap_via_2.25U -> keyswitch:CherryMX_Hotswap_via_2.25U
- SW54: footprint BrownSugar_KBD:CherryMX_Hotswap_via_2.75U -> keyswitch:CherryMX_Hotswap_via_2.75U
- SW55, SW56, SW57, SW60, SW61, SW62: footprint BrownSugar_KBD:CherryMX_Hotswap_via_1.25U -> keyswitch:CherryMX_Hotswap_via_1.25U
- SW58, SW59: footprint BrownSugar_KBD:CherryMX_Hotswap_via_3U -> keyswitch:CherryMX_Hotswap_via_3U
- renumbered Reset to SW1

Commit message: wared
Parts:
- removed the REF** at (223.8, 166.7)
- removed the REF** at (166.7, 166.7)
- removed the REF** at (333.4, 90.5)
- removed the REF** at (331.0, 128.6)
- removed the REF** at (88.1, 147.6)
- removed the REF** at (326.2, 147.6)
- added REF**: Stabilizer, stabilizer:Stabilizer_MX_PCB_Mount_3U, F.Cu at (166.7, 166.7)
- added REF**: Stabilizer, stabilizer:Stabilizer_MX_PCB_Mount_3U, F.Cu at (223.8, 166.7)
- added REF**: Stabilizer, stabilizer:Stabilizer_MX_PCB_Mount_2U, F.Cu at (88.1, 147.6)
- added REF**: Stabilizer, stabilizer:Stabilizer_MX_PCB_Mount_2U, F.Cu at (331.0, 128.6)
- added REF**: Stabilizer, stabilizer:Stabilizer_MX_PCB_Mount_2U, F.Cu at (333.4, 90.5)
- added REF**: Stabilizer, stabilizer:Stabilizer_MX_PCB_Mount_2U, F.Cu at (326.2, 147.6)
- J2: footprint 5077CR-16SMC2-BK-TR:NELTRON_5077CR-16SMC2-BK-TR -> others:Usb_C_NELTRON_5077CR-16SMC2-BK-TR
- SW1: footprint original_library:ResetSW TSHA-T-2.5B2-19SH -> others:ResetSW TSHA-T-2.5B2-19SH
- moved J1 317.1 mm to (69.8, 102.2)
- moved C6 311.4 mm to (69.0, 107.0), turned to 0 degrees
- moved C7 311.4 mm to (69.0, 110.0), turned to 0 degrees
- moved C4 310.8 mm to (69.0, 113.0), turned to 0 degrees
- moved R6 310.3 mm to (69.0, 100.0)
- moved C5 309.6 mm to (69.0, 116.0), turned to 0 degrees
- moved R4 301.6 mm to (78.6, 83.7), turned to -90 degrees
- moved R5 289.2 mm to (92.9, 83.7), turned to 90 degrees
- moved R2 276.8 mm to (106.0, 148.0)
- moved R3 276.8 mm to (103.2, 148.0)
- moved C2 201.4 mm to (180.2, 169.1), turned to 135 degrees
- moved C1 199.7 mm to (179.6, 172.0), turned to -45 degrees
- moved Y1 199.4 mm to (182.6, 166.7), turned to 45 degrees
- moved C3 197.5 mm to (184.9, 164.3), turned to -45 degrees
- moved R1 176.4 mm to (206.0, 167.0), turned to -90 degrees
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Connections:
- SW60 pad 1: col9 -> col8
- U1 pad 1: row0 -> row4
- U1 pad 18: RE_A -> unconnected-(U1-PD0-Pad18)
- U1 pad 19: RE_B -> unconnected-(U1-PD1-Pad19)
- U1 pad 20: col0 -> unconnected-(U1-PD2-Pad20)
- U1 pad 21: col1 -> unconnected-(U1-PD3-Pad21)
- U1 pad 22: col2 -> unconnected-(U1-PD5-Pad22)
- U1 pad 25: col3 -> unconnected-(U1-PD4-Pad25)
- U1 pad 26: col4 -> unconnected-(U1-PD6-Pad26)
- U1 pad 27: col5 -> unconnected-(U1-PD7-Pad27)
- U1 pad 28: col6 -> unconnected-(U1-PB4-Pad28)
- U1 pad 29: col7 -> unconnected-(U1-PB5-Pad29)
- U1 pad 30: col10 -> unconnected-(U1-PB6-Pad30)
- U1 pad 31: col9 -> unconnected-(U1-PC6-Pad31)
- U1 pad 32: col8 -> unconnected-(U1-PC7-Pad32)
- U1 pad 36: row4 -> unconnected-(U1-PF7-Pad36)
- U1 pad 37: row3 -> unconnected-(U1-PF6-Pad37)
- U1 pad 38: col11 -> unconnected-(U1-PF5-Pad38)
- U1 pad 39: col12 -> unconnected-(U1-PF4-Pad39)
- U1 pad 40: row2 -> unconnected-(U1-PF1-Pad40)
- U1 pad 41: row1 -> unconnected-(U1-PF0-Pad41)
- U1 pad 8: col13 -> col0
Routing:
- net row1: track 0.00 -> 285.7 mm
- net GND: track 0.00 -> 280.4 mm, vias 0 -> 4
- net VCC: track 0.00 -> 271.2 mm, vias 0 -> 5
- net row0: track 0.00 -> 265.2 mm
- net row4: track 0.00 -> 264.4 mm
- net row2: track 0.00 -> 246.3 mm
- net row3: track 0.00 -> 218.9 mm
- net col0: track 0.00 -> 210.4 mm, vias 0 -> 2
- net Reset: track 0.00 -> 178.7 mm, vias 0 -> 5
- net Net-(U1-D-): track 0.00 -> 111.3 mm, vias 0 -> 2
- net Net-(U1-D+): track 0.00 -> 108.4 mm, vias 0 -> 2
- net col12: track 0.00 -> 97.3 mm
- net col8: track 0.00 -> 91.0 mm
- net col2: track 0.00 -> 91.0 mm
- net col6: track 0.00 -> 90.0 mm
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Other:
- outline, holes or cut-outs redrawn
