File: my-own-keyboard.kicad_sch (KiCad schematic)
At the start: 142 parts, among them J1 ICSP, J2 5077CR-16SMC2-BK-TR, SW1 Reset SW, SW10 8, SW11 9, SW12 0, SW13 -, SW14 =, SW15 Backspace, SW16 Tab, SW17 Q, SW18 W, SW19 E, SW2 `, SW20 R, SW21 T, SW22 Y, SW23 U, SW24 I, SW25 O, SW26 P, SW27 [, SW28 ], SW29 \, SW3 1, SW30 Capslock, SW31 A, SW32 S, SW33 D, SW34 F, SW35 G, SW36 H, SW37 J, SW38 K, SW39 L, SW4 2, SW40 ;, SW41 ', SW42 Enter, SW43 L-shift, SW44 Z, SW45 X, SW46 C, SW47 V, SW48 B, SW49 N, SW5 3, SW50 M, SW51 ,, SW52 ., SW53 /, SW54 R-shift, SW55 L-Ctrl, SW56 win, SW57 L-Alt, SW58 Space, SW59 Fn, SW6 4, SW60 R-Alt, SW61 Menu, SW62 R-Ctrl, SW63 RotaryEncoder_Switch, SW7 5, SW8 6, SW9 7, U1 ATmega32U4-A, Y1 16MHz

Commit message: updated the directory
Parts:
- D1, D10, D11, D12, D13, D14, D15, D16, D17, D18, D19, D2, D20, D21, D22, D23, D24, D25, D26, D27, D28, D29, D3, D30, D31, D32, D33, D34, D35, D36, D37, D38, D39, D4, D40, D41, D42, D43, D44, D45, D46, D47, D48, D49, D5, D50, D51, D52, D53, D54, D55, D56, D57, D58, D59, D6, D60, D61, D62, D7, D8, D9: footprint kbd:D3_TH_SMD -> others:D3_TH_SMD
- SW10, SW11, SW12, SW13, SW14, SW17, SW18, SW19, SW2, SW20, SW21, SW22, SW23, SW24, SW25, SW26, SW27, SW28, SW3, SW31, SW32, SW33, SW34, SW35, SW36, SW37, SW38, SW39, SW4, SW40, SW41, SW44, SW45, SW46, SW47, SW48, SW49, SW5, SW50, SW51, SW52, SW53, SW6, SW7, SW8, SW9: footprint BrownSugar_KBD:CherryMX_Hotswap_via_1U -> keyswitch:CherryMX_Hotswap_via_1U
- SW15: footprint BrownSugar_KBD:CherryMX_Hotswap_via_2U -> keyswitch:CherryMX_Hotswap_via_2U
- SW16, SW29: footprint BrownSugar_KBD:CherryMX_Hotswap_via_1.5U -> keyswitch:CherryMX_Hotswap_via_1.5U
- SW30: footprint BrownSugar_KBD:CherryMX_Hotswap_via_1.75U -> keyswitch:CherryMX_Hotswap_via_1.75U
- SW42, SW43: footprint BrownSugar_KBD:CherryMX_Hotswap_via_2.25U -> keyswitch:CherryMX_Hotswap_via_2.25U
- SW54: footprint BrownSugar_KBD:CherryMX_Hotswap_via_2.75U -> keyswitch:CherryMX_Hotswap_via_2.75U
- SW55, SW56, SW57, SW60, SW61, SW62: footprint BrownSugar_KBD:CherryMX_Hotswap_via_1.25U -> keyswitch:CherryMX_Hotswap_via_1.25U
- SW58, SW59: footprint BrownSugar_KBD:CherryMX_Hotswap_via_3U -> keyswitch:CherryMX_Hotswap_via_3U

Commit message: wared
Parts:
- J2: footprint 5077CR-16SMC2-BK-TR:NELTRON_5077CR-16SMC2-BK-TR -> others:Usb_C_NELTRON_5077CR-16SMC2-BK-TR
- SW1: footprint original_library:ResetSW TSHA-T-2.5B2-19SH -> others:ResetSW TSHA-T-2.5B2-19SH
Connections:
- net RE_A: no longer U1.18 (PD0)
- net RE_B: no longer U1.19 (PD1)
- net col0: now also U1.8 (PB0); no longer U1.20 (PD2)
- net col1: no longer U1.21 (PD3)
- net col10: no longer U1.30 (PB6)
- net col11: no longer U1.38 (PF5)
- net col12: no longer U1.39 (PF4)
- net col13: no longer U1.8 (PB0)
- net col2: no longer U1.22 (PD5)
- net col3: no longer U1.25 (PD4)
- net col4: no longer U1.26 (PD6)
- net col5: no longer U1.27 (PD7)
- net col6: no longer U1.28 (PB4)
- net col7: no longer U1.29 (PB5)
- net col8: now also SW60.1; no longer U1.32 (PC7)
- net col9: no longer SW60.1, U1.31 (PC6)
- net row0: no longer U1.1 (PE6)
- net row1: no longer U1.41 (PF0)
- net row2: no longer U1.40 (PF1)
- net row3: no longer U1.37 (PF6)
- net row4: now also U1.1 (PE6); no longer U1.36 (PF7)
- no-connect marks 4 -> 3
Other:
- moved on the sheet: D59, SW60
